Commit message: copying codes to github

File: urdfbot_description/urdf/urdfbot_simple.urdf (robot description, URDF)
Before this commit: robot urdfbot, 6 links, 5 joints
Links:
- removed link claw_a_r_link
- removed link claw_b_r_link
- removed link lower_arm_r_link
- removed link upper_arm_r_link
Joints:
- removed joint base_link_to_upper_arm_r_link_joint
- removed joint upper_arm_r_link_to_claw_a_r_link_joint
- removed joint upper_arm_r_link_to_claw_b_r_link_joint
- removed joint upper_arm_r_link_to_lower_arm_r_link_joint
